File: circuitoAzulyOro/circuitoAzulyOro.sch (KiCad schematic (older format))
At the start: 20 parts, among them U1 ATMEGA328PB-AU

Commit message: added FTDI and voltage reg
Parts:
- removed C?: CP, symbol CP
- removed SW?: SW_Push, symbol SW_Push
- added C? (x3): 100nF, symbol C
- added C?: 4.7uF_16V, symbol CP
- added J1: USB, symbol USB_OTG
- added J2: ICSP, symbol Conn_02x03_Odd_Even
- added RP2B, RP2D: 1K, symbol R
- added RXRed, TXGreen: LED, symbol LED
- added U2: FT232RL, Package_SO:SSOP-28_5.3x10.2mm_P0.65mm, symbol FT232RL
- added U?: LM1117-5.0, symbol LM1117-5.0
- C?: value C -> 1uF
- D?: value LED -> PWRGreen
- RP1C: renamed from R?; value R -> 1K
- gave numbers to parts that had none: 1
Connections:
- net labels added: +5VD, VSS
- wire segments 64 -> 137
Other:
- note added: "TODO:\nMOSFET MOTOR CONTROL\nIMU?\nSERVO Headers\n"
- moved on the sheet: C?, D?, F1, RP1A, RP1B, RP1C, RP1D, RP2A, Reset_Button, U1, Y?

Commit message: todo list added
Parts:
- gave numbers to parts that had none: 1
Other:
- note added: "TODO:\nMOSFET MOTOR CONTROL\nIMU?\nBattery holder and conn\nSERVO Headers\ndebugging leds?\nanalog sensor?\nextension connectors for RF/bluetooth module?\n"
- note removed: "TODO:\nMOSFET MOTOR CONTROL\nIMU?\nSERVO Headers\n"
Changed lines of the file:
@@
 	7200 3550 7200 2550
 $Comp
-L LM1117-5.0 U?
+L LM1117-5.0 U3
 U 1 1 5B9A48BB
 P 7700 4200
-F 0 "U?" H 7550 4325 50  0000 C CNN
+F 0 "U3" H 7550 4325 50  0000 C CNN
 F 1 "LM1117-5.0" H 7700 4325 50  0000 L CNN
 F 2 "" H 7700 4200 50  0001 C CNN
@@
 Wire Notes Line
 	7000 4950 7000 3800
-Text Notes 4700 5800 2    60   ~ 0
-TODO:\nMOSFET MOTOR CONTROL\nIMU?\nSERVO Headers\n
+Text Notes 2250 7900 0    197  ~ 0
+TODO:\nMOSFET MOTOR CONTROL\nIMU?\nBattery holder and conn\nSERVO Headers\ndebugging leds?\nanalog sensor?\nextension connectors for RF/bluetooth module?\n
 $EndSCHEMATC
